File: kicad/metronome.kicad_pcb (KiCad board)
At the start: 2 copper layers, 34.5 x 48.8 mm, 26 parts, among them J1 Conn_01x02, J2 Conn_01x02, J3 Conn_01x04, Q1 BS170, U1 LM555xN, U2 4017

Commit message: Update gerber files
Other:
- board text added: "2"
- board text added: "3"
- board text added: "4"
- board text added: "Metronome V1.0, 20-240 bpm by Paavo Palomäki 04/2022"
- board text added: "in"
- board text added: "out"
- board text added: "r"
- board text added: "vcc"
- board text removed: "Metronome V1.0 20-240 bpm by Paavo Palomäki 04/2022"
Changed lines of the file:
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@@
     (fp_line (start 9.95 -2.35) (end -2.45 -2.35) (layer "F.Fab") (width 0.1))
     (fp_line (start -2.45 3.4) (end 9.95 3.4) (layer "F.Fab") (width 0.1))
-    (pad "1" thru_hole roundrect locked (at 0 0 270) (size 1.7 1.95) (drill 0.95) (layers *.Cu *.Mask) (roundrect_rratio 0.147059)
+    (pad "1" thru_hole roundrect locked (at 0 0 270) (size 1.7 1.95) (drill 0.95) (layers *.Cu *.Mask) (roundrect_rratio 0.1470588235)
       (net 23 "Net-(U2-Pad15)") (pinfunction "Pin_1") (pintype "passive"))
     (pad "2" thru_hole oval locked (at 2.5 0 270) (size 1.7 1.95) (drill 0.95) (layers *.Cu *.Mask)
@@
   (gr_arc (start 147 110) (mid 145.974874 112.474874) (end 143.5 113.5) (layer "Edge.Cuts") (width 0.1))
   (gr_arc (start 116 113.5) (mid 113.525126 112.474874) (end 112.5 110) (layer "Edge.Cuts") (width 0.1))
-  (gr_text "100k freqpot" (at 139.75 83.5 90) (layer "B.SilkS")
-    (effects (font (size 1.2 1.2) (thickness 0.3)) (justify right mirror))
-  )
-  (gr_text "gnd" (at 120.5 103.25) (layer "B.SilkS")
-    (effects (font (size 1.2 1.2) (thickness 0.3)) (justify left mirror))
-  )
-  (gr_text "speaker" (at 139.75 91.5 90) (layer "B.SilkS")
-    (effects (font (size 1.2 1.2) (thickness 0.3)) (justify right mirror))
-  )
-  (gr_text "bpm = 60/(0.693(2Ra+Rb+R_freqpot)C)" (at 141.75 73.25 90) (layer "B.SilkS")
-    (effects (font (size 1 1) (thickness 0.25)) (justify left mirror))
-  )
-  (gr_text "rhythm_switch" (at 139.75 105.75 90) (layer "B.SilkS")
-    (effects (font (size 1.2 1.2) (thickness 0.3)) (justify right mirror))
-  )
-  (gr_text "Metronome V1.0\n20-240 bpm\nby Paavo Palomäki\n04/2022" (at 136.5 101.75) (layer "B.SilkS")
+  (gr_text "bpm = 60/(0.693(2Ra+Rb+R_freqpot)C)" (at 143.5 93) (layer "B.SilkS")
     (effects (font (size 0.9 0.9) (thickness 0.225)) (justify left mirror))
   )
-  (gr_text "vin" (at 119.75 100.75) (layer "B.SilkS")
-    (effects (font (size 1.2 1.2) (thickness 0.3)) (justify left mirror))
+  (gr_text "Metronome V1.0, 20-240 bpm\nby Paavo Palomäki 04/2022" (at 140 90.5) (layer "B.SilkS")
+    (effects (font (size 0.9 0.9) (thickness 0.225)) (justify left mirror))
   )
   (gr_text "R_vol" (at 137.75 82.25 90) (layer "F.SilkS")
@@
     (effects (font (size 1.2 1.2) (thickness 0.3)) (justify left))
   )
+  (gr_text "in" (at 141.25 75) (layer "F.SilkS")
+    (effects (font (size 0.9 0.9) (thickness 0.225)) (justify left))
+  )
   (gr_text "100k freqpot" (at 139.75 83.5 90) (layer "F.SilkS")
     (effects (font (size 1.2 1.2) (thickness 0.3)) (justify left))
@@
     (effects (font (size 1.2 1.2) (thickness 0.3)) (justify left))
   )
+  (gr_text "out" (at 140.5 80) (layer "F.SilkS")
+    (effects (font (size 0.9 0.9) (thickness 0.225)) (justify left))
+  )
   (gr_text "10u" (at 135 66.75) (layer "F.SilkS")
     (effects (font (size 1.2 1.2) (thickness 0.3)) (justify left))
@@
     (effects (font (size 1.2 1.2) (thickness 0.3)) (justify left))
   )
+  (gr_text "vcc" (at 140.5 86.5) (layer "F.SilkS")
+    (effects (font (size 0.9 0.9) (thickness 0.225)) (justify left))
+  )
   (gr_text "gnd" (at 117 103.25) (layer "F.SilkS")
-    (effects (font (size 1.2 1.2) (thickness 0.3)) (justify left))
-  )
-  (gr_text "LM555" (at 125.26 85 90) (layer "F.SilkS")
+    (effects (font (size 0.9 0.9) (thickness 0.225)) (justify left))
+  )
+  (gr_text "r" (at 141.5 95.5) (layer "F.SilkS")
+    (effects (font (size 0.9 0.9) (thickness 0.225)) (justify left))
+  )
+  (gr_text "LM555" (at 125.26 83.5 90) (layer "F.SilkS")
     (effects (font (size 1.2 1.2) (thickness 0.3)) (justify left))
   )
@@
     (effects (font (size 1.2 1.2) (thickness 0.3)) (justify left))
   )
-  (gr_text "CD4017BE" (at 120.25 91.5) (layer "F.SilkS")
-    (effects (font (size 1.2 1.2) (thickness 0.3)) (justify left))
+  (gr_text "CD4017BE" (at 124 91.5) (layer "F.SilkS")
+    (effects (font (size 1.2 1.2) (thickness 0.3)) (justify left))
+  )
+  (gr_text "gnd" (at 140.5 89) (layer "F.SilkS")
+    (effects (font (size 0.9 0.9) (thickness 0.225)) (justify left))
   )
   (gr_text "5k6" (at 124 67.75) (layer "F.SilkS")
@@
   )
   (gr_text "vin" (at 117 100.75) (layer "F.SilkS")
-    (effects (font (size 1.2 1.2) (thickness 0.3)) (justify left))
+    (effects (font (size 0.9 0.9) (thickness 0.225)) (justify left))
   )
   (gr_text "led_N" (at 130.5 112.25) (layer "F.SilkS")
     (effects (font (size 1.2 1.2) (thickness 0.3)) (justify left))
   )
+  (gr_text "4" (at 141.5 98) (layer "F.SilkS")
+    (effects (font (size 0.9 0.9) (thickness 0.225)) (justify left))
+  )
   (gr_text "10k" (at 115 94 90) (layer "F.SilkS")
     (effects (font (size 1.2 1.2) (thickness 0.3)) (justify left))
   )
-  (gr_text "bpm = 60/(0.693(2Ra+Rb+R_freqpot)C)" (at 141.75 104.75 90) (layer "F.SilkS")
-    (effects (font (size 1 1) (thickness 0.25)) (justify left))
+  (gr_text "2" (at 141.5 103) (layer "F.SilkS")
+    (effects (font (size 0.9 0.9) (thickness 0.225)) (justify left))
+  )
+  (gr_text "in" (at 141.25 77.5) (layer "F.SilkS")
+    (effects (font (size 0.9 0.9) (thickness 0.225)) (justify left))
   )
   (gr_text "680" (at 124 71) (layer "F.SilkS")
@@
     (effects (font (size 1.2 1.2) (thickness 0.3)) (justify left))
   )
+  (gr_text "3" (at 141.5 100.5) (layer "F.SilkS")
+    (effects (font (size 0.9 0.9) (thickness 0.225)) (justify left))
+  )
   (gr_text "Ra" (at 127.75 67.75) (layer "F.SilkS")
