File: kicad/metronome.kicad_sch (KiCad schematic)
At the start: 26 parts, among them J1 Conn_01x02, J2 Conn_01x02, Q1 BS170, U1 LM555xN, U2 4017

Commit message: Update gerber files
Parts:
- J3: value (none) -> Conn_01x04; footprint (none) -> Connector_JST:JST_XH_B4B-XH-A_1x04_P2.50mm_Vertical
Changed lines of the file:
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@@
     (in_bom yes) (on_board yes) (fields_autoplaced)
     (property "Reference" "J3" (id 0) (at 96.52 123.19 90))
-    (property "Value" "" (id 1) (at 96.52 125.73 90))
-    (property "Footprint" "" (id 2) (at 95.25 129.54 0)
+    (property "Value" "Conn_01x04" (id 1) (at 96.52 125.73 90))
+    (property "Footprint" "Connector_JST:JST_XH_B4B-XH-A_1x04_P2.50mm_Vertical" (id 2) (at 95.25 129.54 0)
       (effects (font (size 1.27 1.27)) hide)
     )
